Commit message: ompl planning for reachy2

File: reachy_description/urdf/arm.urdf.xacro (robot description, xacro)
@@ -22,4 +22,6 @@
     <xacro:property name="arm_offset_z" value="0.0" />
     <!-- Define robot model argument -->
+    <xacro:property name="arm_offset_yaw" value="0.17453292519943295" /> <!-- 10 degrees -->
+    <xacro:property name="arm_offset_roll" value="-0.2617993877991494" /> <!-- -15 degrees -->
     <!-- Check if the robot model is 'beta' -->
     <xacro:if value="${robot_model == 'beta'}">
