Commit message: works on hardware!

File: reachy_description/urdf/arm.urdf.xacro (robot description, xacro)
@@ -60,5 +60,5 @@
     <xacro:if value="${side == 'left'}">
       <xacro:property name="reflect" value="-1" />
-      <xacro:property name="min_shoulder_roll" value="-0.0" />
+      <xacro:property name="min_shoulder_roll" value="-${pi}" />
       <xacro:property name="max_shoulder_roll" value="${pi}" />
       <xacro:property name="shoulder_axis1_inverted" value="0" />
@@ -70,5 +70,5 @@
       <xacro:property name="reflect" value="1" />
       <xacro:property name="min_shoulder_roll" value="-${pi}" />
-      <xacro:property name="max_shoulder_roll" value="0.0" />
+      <xacro:property name="max_shoulder_roll" value="${pi}" />
       <xacro:property name="shoulder_axis1_inverted" value="1" />
       <xacro:property name="shoulder_axis2_inverted" value="0" />
@@ -174,15 +174,15 @@
     <!-- <link name="${prefix}_elbow_forearm_link"> -->
     <!--   <visual> -->
-    <!--   	<origin xyz="0 0 0" rpy="0 0 0"/> -->
-    <!--   	<geometry> -->
-    <!-- 	  <mesh filename="package://arm_description/meshes/Orbita2D_forearm.dae" /> -->
-    <!--   	</geometry> -->
+    <!--        <origin xyz="0 0 0" rpy="0 0 0"/> -->
+    <!--        <geometry> -->
+    <!--          <mesh filename="package://arm_description/meshes/Orbita2D_forearm.dae" /> -->
+    <!--        </geometry> -->
     <!--   </visual> -->
     <!--   <inertial> -->
-    <!--   	<origin xyz="0.00092892 -0.00254548 0.14021211" rpy="0 0 0"/> -->
-    <!-- 	<mass value="0.90719109"/> -->
-    <!-- 	 <inertia ixx="0.00428278" ixy="-0.00000203" ixz="0.00011755" -->
-    <!-- 		  iyx="-0.00000203" iyy="0.0044585" iyz="-0.00004915" -->
-    <!-- 		  izx="0.00011755" izy="-0.00004915" izz="0.00047615"/> -->
+    <!--        <origin xyz="0.00092892 -0.00254548 0.14021211" rpy="0 0 0"/> -->
+    <!--        <mass value="0.90719109"/> -->
+    <!--         <inertia ixx="0.00428278" ixy="-0.00000203" ixz="0.00011755" -->
+    <!--                  iyx="-0.00000203" iyy="0.0044585" iyz="-0.00004915" -->
+    <!--                  izx="0.00011755" izy="-0.00004915" izz="0.00047615"/> -->
     <!--   </inertial> -->
     <!-- </link> -->
