Commit message: Fix shoulder roll joint limits and audit joint limit consistency
The URDF bounded *_shoulder_roll at exactly 0.0 (left: [-0.0, pi],
right: [-pi, 0.0]) while the Orbita2D software limits allow +/-0.55 rad
and the mechanical stops sit at +/-0.61. Since Orbita2dSystem::read()
publishes the measured orientation unclamped, joint_states routinely
reported values up to 0.55 rad outside the declared limits - well past
MoveIt's start_state_max_bounds_error of 0.1 - causing planning to fail
on the real robot.

Upstream fixed this in reachy2_core 04f3b11 (released in v1.7.6); this
fork branched from the v1.7.5 line and never picked it up, which is why
the 1.7.5.9 image still carries the old value. Align with upstream by
setting the bound to +/-0.51, matching the fake shoulder configs too,
and update the stale reachy2.urdf snapshot accordingly.

Also add docs/joint_limits_audit.md covering the remaining mismatches
that cannot be fixed from this repository (Orbita3D wrist/neck bounds of
+/-0.35 rad vs a 42.5 degree mechanical cone with no software limit, the
+/-10000 rad placeholder limits on shoulder pitch / elbow yaw, and the
fake elbow config exceeding the URDF bound in simulation).

Co-Authored-By: Claude Opus 5 <noreply@anthropic.com>
Claude-Session: https://claude.ai/code/session_01PUomLVjPuJFLnHDNzkiU4t

File: reachy_description/urdf/arm.urdf.xacro (robot description, xacro)
@@ -60,5 +60,5 @@
     <xacro:if value="${side == 'left'}">
       <xacro:property name="reflect" value="-1" />
-      <xacro:property name="min_shoulder_roll" value="-0.0" />
+      <xacro:property name="min_shoulder_roll" value="-0.51" />
       <xacro:property name="max_shoulder_roll" value="${pi}" />
       <xacro:property name="shoulder_axis1_inverted" value="0" />
@@ -70,5 +70,5 @@
       <xacro:property name="reflect" value="1" />
       <xacro:property name="min_shoulder_roll" value="-${pi}" />
-      <xacro:property name="max_shoulder_roll" value="0.0" />
+      <xacro:property name="max_shoulder_roll" value="0.51" />
       <xacro:property name="shoulder_axis1_inverted" value="1" />
       <xacro:property name="shoulder_axis2_inverted" value="0" />

File: reachy_description/urdf/reachy2.urdf (robot description, URDF)
Before this commit: robot reachy2, 100 links, 99 joints
Joints:
- joint l_shoulder_roll: limit lower=-0.0 upper=3.141592653589793 effort=1000.0 velocity=100.0 -> lower=-0.51 upper=3.141592653589793 effort=1000.0 velocity=100.0
- joint r_shoulder_roll: limit lower=-3.141592653589793 upper=0.0 effort=1000.0 velocity=100.0 -> lower=-3.141592653589793 upper=0.51 effort=1000.0 velocity=100.0
