Commit message: working camera with point cloud data

File: reachy_description/urdf/reachy.urdf.xacro (robot description, xacro)
@@ -578,11 +578,11 @@
   </link>
   <joint name="depth_cam_l_optical_joint" type="fixed">
-    <origin xyz="0.058 0.025 -0.03" rpy="${radians(-47.5-90.0)} 0.0 ${-pi/2}" />
-    <parent link="torso" />
+    <origin xyz="0.058 0.025 -0.03" rpy="${-pi/2} 0.0 ${-pi/2}" />
+    <parent link="head_tip" />
     <child link="depth_cam_l_optical" />
   </joint>
   <joint name="depth_cam_l_frame_joint" type="fixed">
-    <origin xyz="0.058 0.025 -0.03" rpy="0.0 ${radians(47.5)} 0.0" />
-    <parent link="torso" />
+    <origin xyz="0.058 0.025 -0.03" rpy="0.0 0.0 0.0" />
+    <parent link="head_tip" />
     <child link="depth_cam_l_frame" />
   </joint>
@@ -609,16 +609,16 @@
   </link>
   <joint name="depth_cam_rgb_optical_joint" type="fixed">
-    <origin xyz="0.058 0.0155 -0.03" rpy="${radians(-47.5-90.0)} 0.0 ${-pi/2}" />
-    <parent link="torso" />
+    <origin xyz="0.058 0.0155 -0.03" rpy="${-pi/2} 0.0 ${-pi/2}" />
+    <parent link="head_tip" />
     <child link="depth_cam_rgb_optical" />
   </joint>
   <joint name="depth_cam_rgb_optical_frame_joint" type="fixed">
-    <origin xyz="0.058 0.0155 -0.03" rpy="${radians(-47.5-90.0)} 0.0 ${-pi/2}" />
-    <parent link="torso" />
+    <origin xyz="0.058 0.0155 -0.03" rpy="${-pi/2} 0.0 ${-pi/2}" />
+    <parent link="head_tip" />
     <child link="depth_cam_rgb_optical_frame" />
   </joint>
   <joint name="depth_cam_rgb_frame_joint" type="fixed">
-    <origin xyz="0.058 0.0155 -0.03" rpy="0.0 ${radians(47.5)} 0.0" />
-    <parent link="torso" />
+    <origin xyz="0.058 0.0155 -0.03" rpy="0.0 0.0 0.0" />
+    <parent link="head_tip" />
     <child link="depth_cam_rgb_frame" />
   </joint>
@@ -638,11 +638,11 @@
   </link>
   <joint name="depth_cam_r_optical_joint" type="fixed">
-    <origin xyz="0.058 -0.025 -0.03" rpy="${radians(-47.5-90.0)} 0.0 ${-pi/2}" />
-    <parent link="torso" />
+    <origin xyz="0.058 -0.025 -0.03" rpy="${-pi/2} 0.0 ${-pi/2}" />
+    <parent link="head_tip" />
     <child link="depth_cam_r_optical" />
   </joint>
   <joint name="depth_cam_r_frame_joint" type="fixed">
-    <origin xyz="0.058 -0.025 -0.03" rpy="0.0 ${radians(47.5)} 0.0 " />
-    <parent link="torso" />
+    <origin xyz="0.058 -0.025 -0.03" rpy="0.0 0.0 0.0 " />
+    <parent link="head_tip" />
     <child link="depth_cam_r_frame" />
   </joint>

Commit message: add torso camera

File: reachy_description/urdf/reachy.urdf.xacro (robot description, xacro)
@@ -623,4 +623,81 @@
     <child link="depth_cam_rgb_frame" />
   </joint>
+  <!-- Torso camera (forward-facing RGB camera mounted on the chest) -->
+  <link name="torso_camera">
+    <inertial>
+      <mass value="1e-5" />
+      <origin xyz="0 0 0" rpy="0 0 0" />
+      <inertia ixx="1e-6" ixy="0" ixz="0" iyy="1e-6" iyz="0" izz="1e-6" />
+    </inertial>
+  </link>
+  <joint name="torso_camera_fixed" type="fixed">
+    <origin xyz="0.05 0 0.0" rpy="0.0 0.0 0.0" />
+    <parent link="torso" />
+    <child link="torso_camera" />
+  </joint>
+  <link name="torso_camera_optical">
+    <inertial>
+      <origin xyz="0.0 0.0 0.0" rpy="0.0 0.0 0.0" />
+      <mass value="0.001" />
+      <inertia ixx="1.0e-6" ixy="1.0e-8" ixz="1.0e-8" iyy="1.0e-6" iyz="1.0e-8" izz="1.0e-6" />
+    </inertial>
+  </link>
+  <joint name="torso_camera_optical_joint" type="fixed">
+    <!-- standard optical-frame rotation so the gazebo camera image
+         aligns with the link it originates from -->
+    <origin xyz="0 0 0" rpy="${-pi/2.0} 0 ${-pi/2.0}" />
+    <parent link="torso_camera" />
+    <child link="torso_camera_optical" />
+  </joint>
+  <xacro:if value="$(arg use_gazebo)">
+    <gazebo reference="torso_camera">
+      <sensor type="depth" name="torso_camera">
+        <always_on>1</always_on>
+        <update_rate>30</update_rate>
+        <pose>0 0 0 0 0 0</pose>
+        <camera name="torso_camera">
+          <horizontal_fov>${radians(80)}</horizontal_fov>
+          <image>
+            <width>960</width>
+            <height>720</height>
+            <format>R8G8B8</format>
+          </image>
+          <clip>
+            <near>0.1</near>
+            <far>8.0</far>
+          </clip>
+          <distortion>
+            <k1>0.0</k1>
+            <k2>0.0</k2>
+            <k3>0.0</k3>
+            <p1>0.0</p1>
+            <p2>0.0</p2>
+            <center>0.5 0.5</center>
+          </distortion>
+          <noise>
+            <type>gaussian</type>
+            <mean>0.0</mean>
+            <stddev>0.007</stddev>
+          </noise>
+        </camera>
+        <plugin name="torso_camera_controller" filename="libgazebo_ros_camera.so">
+          <ros>
+            <namespace>/torso_camera</namespace>
+            <remapping>torso_camera/image_raw:=color/image_raw</remapping>
+            <remapping>torso_camera/image_raw/compressed:=color/image_raw/compressed</remapping>
+            <remapping>torso_camera/camera_info:=color/camera_info</remapping>
+            <remapping>torso_camera/image_depth:=depth/image_raw</remapping>
+            <remapping>torso_camera/camera_info_depth:=depth/camera_info</remapping>
+            <remapping>torso_camera/points:=depth/points</remapping>
+          </ros>
+          <camera_name>torso_camera</camera_name>
+          <frame_name>torso_camera_optical</frame_name>
+          <hack_baseline>0.0</hack_baseline>
+          <min_depth>0.1</min_depth>
+          <max_depth>8.0</max_depth>
+        </plugin>
+      </sensor>
+    </gazebo>
+  </xacro:if>
   <link name="depth_cam_r_optical">
     <inertial>
