Commit message: reachy2.urdf: latest upstream joint limits (Orbita3D roll/pitch +-0.70, shoulder roll 0.51)
The generated snapshot still carried the limits of orbita3d_control v1.1.5 and the pre-fix
arm xacro. Bring it in line with the current upstream sources:

- neck_roll/neck_pitch and {l,r}_wrist_roll/{l,r}_wrist_pitch: -0.35/0.35 -> -0.70/0.70 rad,
  as orbita3d_description declares since pollen-robotics/orbita3d_control da373b8 ("Update
  angle limits of O3D.", v1.1.6, 2026-01-06). The Orbita3D reaches a ~42.5 deg cone.
- r_shoulder_roll upper 0.0 -> 0.51, l_shoulder_roll lower 0.0 -> -0.51, matching
  arm.urdf.xacro min/max_shoulder_roll after pollen-robotics/reachy2_core 04f3b11
  ("Fix shoulder roll limits.", merged here with pollen/develop).

Co-Authored-By: Claude Opus 5 <noreply@anthropic.com>

File: reachy_description/urdf/reachy2.urdf (robot description, URDF)
Before this commit: robot reachy2, 100 links, 99 joints
Joints:
- joint l_shoulder_roll: limit lower=-0.0 upper=3.141592653589793 effort=1000.0 velocity=100.0 -> lower=-0.51 upper=3.141592653589793 effort=1000.0 velocity=100.0
- joint l_wrist_pitch: limit lower=-0.35 upper=0.35 effort=1000.0 velocity=100.0 -> lower=-0.70 upper=0.70 effort=1000.0 velocity=100.0
- joint l_wrist_roll: limit lower=-0.35 upper=0.35 effort=1000.0 velocity=100.0 -> lower=-0.70 upper=0.70 effort=1000.0 velocity=100.0
- joint neck_pitch: limit lower=-0.35 upper=0.35 effort=1000.0 velocity=100.0 -> lower=-0.70 upper=0.70 effort=1000.0 velocity=100.0
- joint neck_roll: limit lower=-0.35 upper=0.35 effort=1000.0 velocity=100.0 -> lower=-0.70 upper=0.70 effort=1000.0 velocity=100.0
- joint r_shoulder_roll: limit lower=-3.141592653589793 upper=0.0 effort=1000.0 velocity=100.0 -> lower=-3.141592653589793 upper=0.51 effort=1000.0 velocity=100.0
- joint r_wrist_pitch: limit lower=-0.35 upper=0.35 effort=1000.0 velocity=100.0 -> lower=-0.70 upper=0.70 effort=1000.0 velocity=100.0
- joint r_wrist_roll: limit lower=-0.35 upper=0.35 effort=1000.0 velocity=100.0 -> lower=-0.70 upper=0.70 effort=1000.0 velocity=100.0
