Commit message: Align camera descriptions and isolate hardware launch modes

File: reachy_description/urdf/head.urdf.xacro (robot description, xacro)
@@ -378,14 +378,8 @@
         </sensor>
       </gazebo>
-      <!-- Head ToF depth camera (Luxonis ToF 33D on the real robot).
-           Publishes into the same /teleop_camera/depth/... namespace and the
-           same tof_camera_optical frame as the physical robot, so the GP-SDF
-           config is identical between sim, bag playback and hardware.
-           horizontal_fov 1.2207509 rad is chosen so gazebo's derived intrinsics
-           match the real ToF: fx = (width/2)/tan(hfov/2) = 320/tan(0.6103755)
-           = 457.0 px, and with square pixels fy = 457.0, cx = 320, cy = 240.
-           (The bag's recorded camera_info reports fy = 376.7, which is a known
-           placeholder — see kernel_sdf_keti/config/reachy/README.md.)
-           Range 0.1-6 m matches depth_frame.yaml's valid_range. -->
+      <!-- Head ToF stream compatibility ported from ERL 01b329a.
+           Intrinsics, noise and range are simulation approximations, not verified
+           calibration of this robot. Compare raw/rectified CameraInfo before use.
+           hfov=1.2207509 at 640x480 gives fx=fy=457.484 px (square pixels). -->
       <xacro:if value="$(arg depth_camera)">
         <gazebo reference="tof_camera">

File: reachy_description/urdf/reachy.urdf.xacro (robot description, xacro)
@@ -578,11 +578,11 @@
   </link>
   <joint name="depth_cam_l_optical_joint" type="fixed">
-    <origin xyz="0.058 0.025 -0.03" rpy="${-pi/2} 0.0 ${-pi/2}" />
-    <parent link="head_tip" />
+    <origin xyz="0.058 0.025 -0.03" rpy="${radians(-47.5-90.0)} 0.0 ${-pi/2}" />
+    <parent link="torso" />
     <child link="depth_cam_l_optical" />
   </joint>
   <joint name="depth_cam_l_frame_joint" type="fixed">
-    <origin xyz="0.058 0.025 -0.03" rpy="0.0 0.0 0.0" />
-    <parent link="head_tip" />
+    <origin xyz="0.058 0.025 -0.03" rpy="0.0 ${radians(47.5)} 0.0" />
+    <parent link="torso" />
     <child link="depth_cam_l_frame" />
   </joint>
@@ -609,16 +609,16 @@
   </link>
   <joint name="depth_cam_rgb_optical_joint" type="fixed">
-    <origin xyz="0.058 0.0155 -0.03" rpy="${-pi/2} 0.0 ${-pi/2}" />
-    <parent link="head_tip" />
+    <origin xyz="0.058 0.0155 -0.03" rpy="${radians(-47.5-90.0)} 0.0 ${-pi/2}" />
+    <parent link="torso" />
     <child link="depth_cam_rgb_optical" />
   </joint>
   <joint name="depth_cam_rgb_optical_frame_joint" type="fixed">
-    <origin xyz="0.058 0.0155 -0.03" rpy="${-pi/2} 0.0 ${-pi/2}" />
-    <parent link="head_tip" />
+    <origin xyz="0.058 0.0155 -0.03" rpy="${radians(-47.5-90.0)} 0.0 ${-pi/2}" />
+    <parent link="torso" />
     <child link="depth_cam_rgb_optical_frame" />
   </joint>
   <joint name="depth_cam_rgb_frame_joint" type="fixed">
-    <origin xyz="0.058 0.0155 -0.03" rpy="0.0 0.0 0.0" />
-    <parent link="head_tip" />
+    <origin xyz="0.058 0.0155 -0.03" rpy="0.0 ${radians(47.5)} 0.0" />
+    <parent link="torso" />
     <child link="depth_cam_rgb_frame" />
   </joint>
@@ -730,11 +730,11 @@
   </link>
   <joint name="depth_cam_r_optical_joint" type="fixed">
-    <origin xyz="0.058 -0.025 -0.03" rpy="${-pi/2} 0.0 ${-pi/2}" />
-    <parent link="head_tip" />
+    <origin xyz="0.058 -0.025 -0.03" rpy="${radians(-47.5-90.0)} 0.0 ${-pi/2}" />
+    <parent link="torso" />
     <child link="depth_cam_r_optical" />
   </joint>
   <joint name="depth_cam_r_frame_joint" type="fixed">
-    <origin xyz="0.058 -0.025 -0.03" rpy="0.0 0.0 0.0 " />
-    <parent link="head_tip" />
+    <origin xyz="0.058 -0.025 -0.03" rpy="0.0 ${radians(47.5)} 0.0 " />
+    <parent link="torso" />
     <child link="depth_cam_r_frame" />
   </joint>

File: reachy_description/urdf/reachy2.urdf (robot description, URDF)
Before this commit: robot reachy2, 100 links, 99 joints
Links:
- added link torso_camera, mass 1e-5
- added link torso_camera_link, mass 0.001
- added link torso_camera_optical, mass 0.001
- link antenna_left_link: geometry visual mesh filename=package://reachy_description/meshes/head_antenna_visual.dae
- link antenna_right_link: geometry visual mesh filename=package://reachy_description/meshes/head_antenna_visual.dae
- link base_link: geometry collision cylinder length=0.19 radius=0.245; visual mesh filename=package://reachy_description/meshes/mobile_base_visual.dae
- link head: geometry collision mesh filename=package://reachy_description/meshes/head_collider.dae; visual mesh filename=package://reachy_description/meshes/head_visual.dae
- link l_elbow_arm_link: geometry collision mesh filename=package://reachy_description/meshes/upper_arm_collider.dae; visual mesh filename=package://reachy_description/meshes/upper_arm_visual.dae
- link l_elbow_first_link: geometry visual mesh filename=package://orbita2d_description/meshes/2D_sphere_visual.dae
- link l_elbow_forearm_link: geometry collision mesh filename=package://reachy_description/meshes/forearm_collider.dae; visual mesh filename=package://reachy_description/meshes/forearm_visual.dae
- link l_hand_distal_link: geometry collision mesh filename=package://dynamixel_description/meshes/pincette_distal_coll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; visual mesh filename=package://dynamixel_description/meshes/pincette_distal.dae
- link l_hand_distal_mimic_link: geometry collision mesh filename=package://dynamixel_description/meshes/pincette_distal_coll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; visual mesh filename=package://dynamixel_description/meshes/pincette_distal.dae
- link l_hand_palm_link: geometry collision mesh filename=package://dynamixel_description/meshes/pincette_base_collid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; visual mesh filename=package://dynamixel_description/meshes/pincette_right_visua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
- link l_hand_proximal_link: geometry collision mesh filename=package://dynamixel_description/meshes/pincette_proximal_co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; visual mesh filename=package://dynamixel_description/meshes/pincette_proximal_vi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
- link l_hand_proximal_mimic_link: geometry collision mesh filename=package://dynamixel_description/meshes/pincette_proximal_co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; visual mesh filename=package://dynamixel_description/meshes/pincette_proximal_vi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
- link l_shoulder_first_link: geometry visual mesh filename=package://orbita2d_description/meshes/2D_sphere_visual.dae
- link r_elbow_arm_link: geometry collision mesh filename=package://reachy_description/meshes/upper_arm_collider.dae; visual mesh filename=package://reachy_description/meshes/upper_arm_visual.dae
- link r_elbow_first_link: geometry visual mesh filename=package://orbita2d_description/meshes/2D_sphere_visual.dae
- link r_elbow_forearm_link: geometry collision mesh filename=package://reachy_description/meshes/forearm_collider.dae; visual mesh filename=package://reachy_description/meshes/forearm_visual.dae
- link r_hand_distal_link: geometry collision mesh filename=package://dynamixel_description/meshes/pincette_distal_coll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; visual mesh filename=package://dynamixel_description/meshes/pincette_distal.dae
- link r_hand_distal_mimic_link: geometry collision mesh filename=package://dynamixel_description/meshes/pincette_distal_coll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; visual mesh filename=package://dynamixel_description/meshes/pincette_distal.dae
- link r_hand_palm_link: geometry collision mesh filename=package://dynamixel_description/meshes/pincette_base_collid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; visual mesh filename=package://dynamixel_description/meshes/pincette_right_visua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
- link r_hand_proximal_link: geometry collision mesh filename=package://dynamixel_description/meshes/pincette_proximal_co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; visual mesh filename=package://dynamixel_description/meshes/pincette_proximal_vi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
- link r_hand_proximal_mimic_link: geometry collision mesh filename=package://dynamixel_description/meshes/pincette_proximal_co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; visual mesh filename=package://dynamixel_description/meshes/pincette_proximal_vi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
- link r_shoulder_first_link: geometry visual mesh filename=package://orbita2d_description/meshes/2D_sphere_visual.dae
- link torso: geometry collision mesh filename=package://reachy_description/meshes/torso_collider.dae; visual mesh filename=package://reachy_description/meshes/torso_visual.dae
Joints:
- added joint torso_camera_fixed: type fixed, parent torso, child torso_camera, origin xyz=0.05 0 0.0 rpy=0.0 0.0 0.0
- added joint torso_camera_link_joint: type fixed, parent torso_camera, child torso_camera_link, origin xyz=0 0 0 rpy=0 0 0
- added joint torso_camera_optical_joint: type fixed, parent torso_camera, child torso_camera_optical, origin xyz=0 0 0 rpy=-1.5707963267948966 0 -1.5707963267948966
- joint depth_cam_l_frame_joint: origin xyz=0.058 0.025 -0.03 rpy=0.0 0.0 0.0 -> xyz=0.058 0.025 -0.03 rpy=0.0 0.8290313946973066 0.0; parent head_tip -> torso
- joint depth_cam_l_optical_joint: origin xyz=0.058 0.025 -0.03 rpy=-1.5707963267948966 0.0 -1.5707963267948966 -> xyz=0.058 0.025 -0.03 rpy=-2.399827721492203 0.0 -1.5707963267948966; parent head_tip -> torso
- joint depth_cam_r_frame_joint: origin xyz=0.058 -0.025 -0.03 rpy=0.0 0.0 0.0  -> xyz=0.058 -0.025 -0.03 rpy=0.0 0.8290313946973066 0.0 ; parent head_tip -> torso
- joint depth_cam_r_optical_joint: origin xyz=0.058 -0.025 -0.03 rpy=-1.5707963267948966 0.0 -1.5707963267948966 -> xyz=0.058 -0.025 -0.03 rpy=-2.399827721492203 0.0 -1.5707963267948966; parent head_tip -> torso
- joint depth_cam_rgb_frame_joint: origin xyz=0.058 0.0155 -0.03 rpy=0.0 0.0 0.0 -> xyz=0.058 0.0155 -0.03 rpy=0.0 0.8290313946973066 0.0; parent head_tip -> torso
- joint depth_cam_rgb_optical_frame_joint: origin xyz=0.058 0.0155 -0.03 rpy=-1.5707963267948966 0.0 -1.5707963267948966 -> xyz=0.058 0.0155 -0.03 rpy=-2.399827721492203 0.0 -1.5707963267948966; parent head_tip -> torso
- joint depth_cam_rgb_optical_joint: origin xyz=0.058 0.0155 -0.03 rpy=-1.5707963267948966 0.0 -1.5707963267948966 -> xyz=0.058 0.0155 -0.03 rpy=-2.399827721492203 0.0 -1.5707963267948966; parent head_tip -> torso
